File: Main Board/lib/od-aws.brd (EAGLE design)
At the start: 139.7 x 106.3 mm, 7 parts

Commit message: update all board
Parts:
- moved POWER 89.9 mm to (10.2, 73.7), turned to 270 degrees
- moved DFROBOT 40.7 mm to (58.4, 8.89), turned to 180 degrees
- moved NET 35.9 mm to (71.1, 73.7), turned to 90 degrees
- moved U$3 19.2 mm to (67.3, 27.9)
- moved U$1 19.1 mm to (6.35, 61.0)
- moved ADDON 11.5 mm to (72.4, 8.89), turned to 180 degrees
- moved U$2 6.35 mm to (76.2, 62.2), flipped to the bottom
Connections:
- removed net 3V: U$1.3V31
- new net +3V3: U$1.3V31, U$3.13
- net +5V: no longer U$3.13
Routing:
- net +3V3: track 0.00 -> 86.1 mm
- net DFTX: track 97.5 -> 55.9 mm, vias 0 -> 1
- net SIMRST: track 35.9 -> 67.9 mm
- net PE: track 185.2 -> 159.1 mm, vias 0 -> 1
- net SIMRX: track 53.1 -> 75.3 mm
- net SIMTX: track 51.4 -> 73.5 mm
- net DFRX: track 83.7 -> 62.0 mm
- net LORANET: track 36.5 -> 57.3 mm
- net SIMNET: track 31.8 -> 15.9 mm
- net MOSI: track 80.8 -> 70.9 mm
- net DHT: track 27.7 -> 37.0 mm
- net ADDSDA: track 52.6 -> 46.0 mm, vias 0 -> 1
- net ADDSCL: track 56.9 -> 63.3 mm
- net +5V: track 146.0 -> 151.2 mm
- net SCK: track 34.5 -> 37.0 mm
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Other:
- board size 139.7 x 106.3 mm -> 82.5 x 77.5 mm
- board text added: "3.3v"
- board text added: "5v"
- board text added: "dht"
- board text added: "gnd"
- board text added: "gsm"
- board text added: "lora"
- board text added: "made in Indonesia"
- board text added: "rx"
- board text added: "scl"
- board text added: "sda"
- board text added: "tx"
