File: Main Board/lib/od-aws.sch (EAGLE design)
At the start: 7 parts

Commit message: update all board
Connections:
- removed net 3V: U$1.3V1
- new net +3V3: U$1.3V1, U$3.3.3V
- net +5V: no longer U$3.3.3V
Changed lines of the file:
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@@
 <part name="SUPPLY11" library="supply2" library_urn="urn:adsk.eagle:library:372" deviceset="PE" device=""/>
 <part name="SUPPLY12" library="supply2" library_urn="urn:adsk.eagle:library:372" deviceset="PE" device=""/>
-<part name="SUPPLY7" library="supply2" library_urn="urn:adsk.eagle:library:372" deviceset="+5V" device="" value="+3.3V"/>
+<part name="+3V1" library="supply1" library_urn="urn:adsk.eagle:library:371" deviceset="+3V3" device=""/>
+<part name="+3V2" library="supply1" library_urn="urn:adsk.eagle:library:371" deviceset="+3V3" device=""/>
 </parts>
 <sheets>
@@
 <instance part="SUPPLY11" gate="PE" x="106.68" y="83.82" smashed="yes"/>
 <instance part="SUPPLY12" gate="PE" x="129.54" y="60.96" smashed="yes"/>
-<instance part="SUPPLY7" gate="+5V" x="129.54" y="48.26" smashed="yes">
-<attribute name="VALUE" x="127.635" y="51.435" size="1.778" layer="96"/>
+<instance part="+3V1" gate="G$1" x="129.54" y="48.26" smashed="yes">
+<attribute name="VALUE" x="127" y="43.18" size="1.778" layer="96" rot="R90"/>
+</instance>
+<instance part="+3V2" gate="G$1" x="10.16" y="83.82" smashed="yes">
+<attribute name="VALUE" x="7.62" y="78.74" size="1.778" layer="96" rot="R90"/>
 </instance>
 </instances>
@@
 </segment>
 </net>
-<net name="3V" class="0">
-<segment>
-<pinref part="U$1" gate="G$1" pin="3V1"/>
-<wire x1="25.4" y1="81.28" x2="17.78" y2="81.28" width="0.1524" layer="91"/>
-<label x="20.32" y="81.28" size="1.778" layer="95"/>
-</segment>
-</net>
 <net name="+5V" class="0">
 <segment>
@@
 <pinref part="ADDON" gate="A" pin="1"/>
 <wire x1="187.96" y1="22.86" x2="195.58" y2="22.86" width="0.1524" layer="91"/>
-</segment>
-<segment>
-<pinref part="SUPPLY7" gate="+5V" pin="+5V"/>
-<pinref part="U$3" gate="G$1" pin="3.3V"/>
-<wire x1="129.54" y1="45.72" x2="152.4" y2="45.72" width="0.1524" layer="91"/>
 </segment>
 <segment>
@@
 </segment>
 </net>
+<net name="+3V3" class="0">
+<segment>
+<pinref part="U$1" gate="G$1" pin="3V1"/>
+<wire x1="10.16" y1="81.28" x2="25.4" y2="81.28" width="0.1524" layer="91"/>
+<wire x1="25.4" y1="81.28" x2="30.48" y2="81.28" width="0.1524" layer="91"/>
+<junction x="25.4" y="81.28"/>
+<pinref part="+3V2" gate="G$1" pin="+3V3"/>
+</segment>
+<segment>
+<pinref part="+3V1" gate="G$1" pin="+3V3"/>
+<pinref part="U$3" gate="G$1" pin="3.3V"/>
+<wire x1="129.54" y1="45.72" x2="152.4" y2="45.72" width="0.1524" layer="91"/>
+</segment>
+</net>
