File: SecondBoard/lib/STM32_new.brd (EAGLE design)
At the start: 100 x 80 mm, 8 parts, among them U1 RFM95W-868S2, X1 22-23-2021

Commit message: clean code and repository
Parts:
- moved U$3 2.61 mm to (52.1, 71.9)
- moved U$2 2.61 mm to (52.2, 67.7)
- renumbered SV1 to SERIAL, SV2 to I2C, X1 to POWER
Connections:
- net GND renamed WE
- removed net N$19: POWER.1, U$1.5V
- net N$1: now also POWER.1, SERIAL.1, U$1.5V; no longer U$1.3.3V1
- net N$13: no longer SERIAL.1
Routing:
- net N$1: track 46.2 -> 137.5 mm
- net N$13: track 93.6 -> 39.3 mm
- net N$19: track 43.0 -> 0.00 mm
- net N$2: track 130.5 -> 135.3 mm
- net N$11: track 15.3 -> 18.0 mm
- net N$12: track 22.7 -> 25.4 mm
- net N$16: track 57.1 -> 58.6 mm
- net N$17: track 66.7 -> 66.1 mm
Other:
- board size 100 x 80 mm -> 59.1 x 63 mm
- board text added: "ADC"
- board text added: "DAPIS - Sebuah sensor cuaca"
- board text added: "Made in Indonesia"
- board text added: "RX"
- board text added: "SCL"
- board text added: "SDA"
- board text added: "SERIAL"
- board text added: "STM32BlackPIll"
- board text added: "TX"
